Commit message: Update custom_bot.xacro

File: urdf/custom_bot.xacro (robot description, xacro)
@@ -42,10 +42,10 @@
   </joint>
   <joint type="fixed" name="camera_joint">
-    <origin xyz="0.2 0 0.1" rpy="0 0 0"/>
+    <origin xyz="0.3 0 0.1" rpy="0 0 0"/>
     <child link="camera"/>
     <parent link="tower"/>
   </joint>
   <joint type="fixed" name="hokuyo_joint">
-    <origin xyz=".15 0 .2" rpy="0 0 0"/>
+    <origin xyz="0.15 0 0.2" rpy="0 0 0"/>
     <child link="hokuyo"/>
     <parent link="tower"/>

Commit message: Update custom_bot.xacro

File: urdf/custom_bot.xacro (robot description, xacro)
@@ -1,4 +1,5 @@
 <?xml version='1.0'?>
 <robot name="udacity_bot" xmlns:xacro="http://www.ros.org/wiki/xacro">
+  <xacro:property name="M_PI" value="3.1415926535897931" />
   <material name="Blue">
     <color rgba="0.0 0.0 0.8 1.0"/>
@@ -74,27 +75,85 @@
     </visual>
   </link>
+  <joint name="camera_joint" type="fixed">
+    <origin xyz="0.3 0 0" rpy="0 -0.4 0" />
+    <parent link="tower" />
+    <child link="camera" />
+  </joint>
   <link name="camera">
     <inertial>
-      <mass value="0.1"/>
-      <origin xyz="0 0 0" rpy="0 0 0"/>
-      <inertia
-              ixx="1e-6" ixy="0" ixz="0"
-              iyy="1e-6" iyz="0"
-              izz="1e-6"
-      />
-    </inertial>
-    <collision name='camera_collision'>
-      <origin xyz="0 0 0" rpy="0 0 0"/>
-      <geometry>
-        <box size="0.05 0.05 0.05"/>
-      </geometry>
-    </collision>
-    <visual name='camera_visual'>
-      <origin xyz="0 0 0" rpy="0 0 0"/>
-      <geometry>
-        <mesh filename="package://slam_project/meshes/kinect.dae"/>
-      </geometry>
-      <material name="Blue"/>
-    </visual>
+      <mass value="0.01" />
+      <origin xyz="0 0 0" />
+      <inertia ixx="0.001" ixy="0.0" ixz="0.0"
+        iyy="0.001" iyz="0.0"
+        izz="0.001" />
+    </inertial>
+    <visual>
+      <origin xyz=" 0 0 0 " rpy="0 0 0" />
+      <geometry>
+        <mesh filename="package://sweeping_bot/meshes/kinect.dae"/>
+      </geometry>
+    </visual>
+    <collision>
+      <origin xyz="0.0 0.0 0.0" rpy="0 0 0" />
+      <geometry>
+        <box size="0.0730 .2760 0.0720"/>
+      </geometry>
+    </collision>
+  </link>
+  <joint name="camera_depth_joint" type="fixed">
+    <origin xyz="0 0.011 0" rpy="0 0 0" />
+    <parent link="camera" />
+    <child link="camera_depth_frame" />
+  </joint>
+  <link name="camera_depth_frame">
+    <inertial>
+      <mass value="0.01" />
+      <origin xyz="0 0 0" />
+      <inertia ixx="0.001" ixy="0.0" ixz="0.0"
+        iyy="0.001" iyz="0.0"
+        izz="0.001" />
+    </inertial>
+  </link>
+  <joint name="camera_depth_optical_joint" type="fixed">
+    <origin xyz="0 0 0" rpy="${-M_PI/2} 0 ${-M_PI/2}" />
+    <parent link="camera_depth_frame" />
+    <child link="camera_depth_optical_frame" />
+  </joint>
+  <link name="camera_depth_optical_frame">
+    <inertial>
+      <mass value="0.001" />
+      <origin xyz="0 0 0" />
+      <inertia ixx="0.0001" ixy="0.0" ixz="0.0"
+        iyy="0.0001" iyz="0.0"
+        izz="0.0001" />
+    </inertial>
+  </link>
+  <joint name="camera_rgb_joint" type="fixed">
+    <origin xyz="0 -0.012 0" rpy="0 0 0" />
+    <parent link="camera" />
+    <child link="camera_rgb_frame" />
+  </joint>
+  <link name="camera_rgb_frame">
+    <inertial>
+      <mass value="0.001" />
+      <origin xyz="0 0 0" />
+      <inertia ixx="0.0001" ixy="0.0" ixz="0.0"
+        iyy="0.0001" iyz="0.0"
+        izz="0.0001" />
+    </inertial>
+  </link>
+  <joint name="camera_rgb_optical_joint" type="fixed">
+    <origin xyz="0 0 0" rpy="${-M_PI/2} 0 ${-M_PI/2}" />
+    <parent link="camera_rgb_frame" />
+    <child link="camera_rgb_optical_frame" />
+  </joint>
+  <link name="camera_rgb_optical_frame">
+    <inertial>
+      <mass value="0.001" />
+      <origin xyz="0 0 0" />
+      <inertia ixx="0.0001" ixy="0.0" ixz="0.0"
+        iyy="0.0001" iyz="0.0"
+        izz="0.0001" />
+    </inertial>
   </link>
   <link name="tower">

Commit message: Update custom_bot.xacro

File: urdf/custom_bot.xacro (robot description, xacro)
@@ -6,5 +6,5 @@
   </material>
   <material name="Red">
-    <color rgba="0.8 0.0 0.0 1.0"/>
+    <color rgba="0.8 0.s0 0.0 1.0"/>
   </material>
   <material name="Green">
@@ -91,5 +91,5 @@
       <origin xyz=" 0 0 0 " rpy="0 0 0" />
       <geometry>
-        <mesh filename="package://sweeping_bot/meshes/kinect.dae"/>
+        <mesh filename="package://slam_project/meshes/kinect.dae"/>
       </geometry>
     </visual>

Commit message: Update custom_bot.xacro

File: urdf/custom_bot.xacro (robot description, xacro)
@@ -41,9 +41,4 @@
     <parent link="chassis"/>
     <child link="tower" />
-  </joint>
-  <joint type="fixed" name="camera_joint">
-    <origin xyz="0.3 0 0.1" rpy="0 0 0"/>
-    <child link="camera"/>
-    <parent link="tower"/>
   </joint>
   <joint type="fixed" name="hokuyo_joint">
